File: custom_split.kicad_pcb (KiCad board)
At the start: 2 copper layers, 135 x 83.1 mm, 36 parts

Commit message: Routed the keeb!
Parts:
- moved B1 26.2 mm to (280.0, 177.4), turned to 0 degrees
- moved JST1 10.2 mm to (258.1, 162.6)
- moved T1 5.08 mm to (282.7, 149.9)
Routing:
- net GND: track 0.00 -> 670.2 mm
- net P5: track 0.00 -> 136.3 mm
- net P2: track 0.00 -> 123.6 mm
- net P10: track 0.00 -> 113.5 mm, vias 0 -> 1
- net P9: track 0.00 -> 112.3 mm
- net P4: track 0.00 -> 104.5 mm
- net P0: track 0.00 -> 100.3 mm
- net P14: track 0.68 -> 100.2 mm
- net P8: track 0.00 -> 96.7 mm
- net P16: track 0.00 -> 95.2 mm
- net P15: track 0.00 -> 92.7 mm, vias 0 -> 1
- net P3: track 0.00 -> 85.8 mm
- net P1: track 0.00 -> 85.2 mm
- net P18: track 0.00 -> 75.9 mm
- net P20: track 0.00 -> 68.3 mm
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